File: pcb/slotag/slotag_v0p1/slotag_v0p1.kicad_pcb (KiCad board)
At the start: 2 copper layers, 54.6 x 14 mm, 29 parts, among them J1 TC2030-JLINK-NL, P1 CONN_01X03, U1 SOLAR_CELL, U2 AM0805, U3 UPG2422TK, U4 74LVC1G04, U5 74LVC1G175, U6 STM32L051K8T6, U7 74LVC1G175, Y1 Crystal_Small

Commit message: minor cosmetic fixes
Parts:
- removed C5: C_Small, Capacitors_SMD:C_0402
- C3, C6, C7: value C_Small -> 100pF
- C4: value 74pF -> 47pF
- R1, R11: value R_Small -> DNP
- R10, R3, R4, R5, R6, R7, R8, R9: value R_Small -> 47K
- R12: value R_Small -> 11K
- R2: value R_Small -> 0
- moved C3 4.83 mm to (137.7, 78.4)
- moved U3 4.83 mm to (138.2, 80.8)
Connections:
- U3 pad 5: Net-(C5-Pad2) -> Net-(A1-Pad1)
Routing:
- net Net-(C7-Pad2): track 7.35 -> 12.2 mm
- net Net-(C6-Pad2): track 7.43 -> 12.3 mm
- net GND: track 23.2 -> 26.8 mm
- net Net-(A1-Pad1): track 4.38 -> 2.45 mm
- net Net-(C5-Pad2): track 1.80 -> 0.00 mm
Other:
- board text added: "SloTag v0.1 Ben Kempke"
