File: pcb/slotag/slotag_v0p1/slotag_v0p1.sch (KiCad schematic (older format))
At the start: 29 parts, among them J1 TC2030-JLINK-NL, P1 CONN_01X03, U1 SOLAR_CELL, U2 AM0805, U3 UPG2422TK, U4 74LVC1G04, U5 74LVC1G175, U6 STM32L051K8T6, U7 74LVC1G175, Y1 Crystal_Small

Commit message: adding component part numbers
Parts:
- C2: DistPartNo (none) -> 478-6613-1-ND; ManPartNo (none) -> TLNN476M010R6000
- C3, C5, C6, C7: value C_Small -> 100pF; DistPartNo (none) -> 490-7754-1-ND; ManPartNo (none) -> GRM1555C1H101JA01J
- C4: value 74pF -> 47pF; DistPartNo (none) -> 490-5942-1-ND; ManPartNo (none) -> GRM1555C1H470JA01D
- R1, R11: value R_Small -> DNP
- R10, R3, R4, R5, R6, R7, R8, R9: value R_Small -> 47K; DistPartNo (none) -> P47.0KLCT-ND; ManPartNo (none) -> ERJ-2RKF4702X
- R12: value R_Small -> 11K; DistPartNo (none) -> P11.0KLCT-ND; ManPartNo (none) -> ERJ-2RKF1102X
- R2: value R_Small -> 0; DistPartNo (none) -> P0.0JCT-ND; ManPartNo (none) -> ERJ-2GE0R00X
- U1: DistPartNo (none) -> 869-1000-ND; ManPartNo (none) -> AM-1417CA
- U3: DistPartNo (none) -> UPG2422TK-A-ND; ManPartNo (none) -> UPG2422TK-A
- U4: DistPartNo (none) -> 568-1579-1-ND; ManPartNo (none) -> 74LVC1G04GW,125
- U5, U7: DistPartNo (none) -> 568-7761-1-ND; ManPartNo (none) -> 74LVC1G175GW,125
- U6: DistPartNo (none) -> 497-14901-ND; ManPartNo (none) -> STM32L051K8T6
Changed lines of the file:
@@
 LIBS:slocalization
 LIBS:polypoint
+LIBS:slotag_v0p1-cache
 EELAYER 25 0
 EELAYER END
@@
 F 2 "Housings_QFP:LQFP-32_7x7mm_Pitch0.8mm" H 4250 3900 60  0001 C CNN
 F 3 "" H 4250 3900 60  0000 C CNN
+F 4 "STM32L051K8T6" H 3500 3450 60  0001 C CNN "ManPartNo"
+F 5 "497-14901-ND" H 3500 3450 60  0001 C CNN "DistPartNo"
 	1    3500 3450
 	1    0    0    -1
@@
 F 2 "slocalization:MINIMOLD-6" H 9400 2250 60  0001 C CNN
 F 3 "" H 9400 2250 60  0000 C CNN
+F 4 "UPG2422TK-A" H 9400 2250 60  0001 C CNN "ManPartNo"
+F 5 "UPG2422TK-A-ND" H 9400 2250 60  0001 C CNN "DistPartNo"
 	1    9400 2250
 	1    0    0    -1
@@
 F 2 "slocalization:AM-1417" H 2400 1650 60  0001 C CNN
 F 3 "" H 2400 1650 60  0000 C CNN
+F 4 "AM-1417CA" H 2400 1650 60  0001 C CNN "ManPartNo"
+F 5 "869-1000-ND" H 2400 1650 60  0001 C CNN "DistPartNo"
 	1    2400 1650
 	-1   0    0    1
@@
 P 8850 1950
 F 0 "C3" H 8942 1996 50  0000 L CNN
-F 1 "C_Small" H 8942 1904 50  0000 L CNN
+F 1 "100pF" H 8942 1904 50  0000 L CNN
 F 2 "Capacitors_SMD:C_0402" H 8850 1950 60  0001 C CNN
 F 3 "" H 8850 1950 60  0000 C CNN
+F 4 "GRM1555C1H101JA01J" H 8850 1950 60  0001 C CNN "ManPartNo"
+F 5 "490-7754-1-ND" H 8850 1950 60  0001 C CNN "DistPartNo"
 	1    8850 1950
 	1    0    0    -1
@@
 P 10200 2250
 F 0 "C5" V 10150 2150 50  0000 C CNN
-F 1 "C_Small" V 10150 2450 50  0000 C CNN
+F 1 "100pF" V 10150 2450 50  0000 C CNN
 F 2 "Capacitors_SMD:C_0402" H 10200 2250 60  0001 C CNN
 F 3 "" H 10200 2250 60  0000 C CNN
+F 4 "GRM1555C1H101JA01J" V 10200 2250 60  0001 C CNN "ManPartNo"
+F 5 "490-7754-1-ND" V 10200 2250 60  0001 C CNN "DistPartNo"
 	1    10200 2250
 	0    1    1    0
@@
 F 2 "Capacitors_SMD:C_0805" H 3800 1550 60  0001 C CNN
 F 3 "" H 3800 1550 60  0000 C CNN
+F 4 "TLNN476M010R6000" H 3800 1550 60  0001 C CNN "ManPartNo"
+F 5 "478-6613-1-ND" H 3800 1550 60  0001 C CNN "DistPartNo"
 	1    3800 1550
 	1    0    0    -1
@@
 P 4950 2000
 F 0 "C4" V 4900 1850 50  0000 C CNN
-F 1 "74pF" V 4900 2200 50  0000 C CNN
+F 1 "47pF" V 4900 2200 50  0000 C CNN
 F 2 "Capacitors_SMD:C_0402" H 4950 2000 60  0001 C CNN
 F 3 "" H 4950 2000 60  0000 C CNN
+F 4 "GRM1555C1H470JA01D" V 4950 2000 60  0001 C CNN "ManPartNo"
+F 5 "490-5942-1-ND" V 4950 2000 60  0001 C CNN "DistPartNo"
 	1    4950 2000
 	0    1    1    0
@@
 P 7450 2050
 F 0 "R1" V 7400 1900 50  0000 C CNN
-F 1 "R_Small" V 7400 2300 50  0000 C CNN
+F 1 "DNP" V 7400 2250 50  0000 C CNN
 F 2 "Resistors_SMD:R_0402" H 7450 2050 60  0001 C CNN
 F 3 "" H 7450 2050 60  0000 C CNN
@@
 P 7450 2250
 F 0 "R2" V 7400 2100 50  0000 C CNN
-F 1 "R_Small" V 7400 2500 50  0000 C CNN
+F 1 "0" V 7400 2400 50  0000 C CNN
 F 2 "Resistors_SMD:R_0402" H 7450 2250 60  0001 C CNN
 F 3 "" H 7450 2250 60  0000 C CNN
+F 4 "ERJ-2GE0R00X" V 7450 2250 60  0001 C CNN "ManPartNo"
+F 5 "P0.0JCT-ND" V 7450 2250 60  0001 C CNN "DistPartNo"
 	1    7450 2250
 	0    1    1    0
@@
 P 6650 2850
 F 0 "R4" V 6600 2700 50  0000 C CNN
-F 1 "R_Small" V 6600 3100 50  0000 C CNN
+F 1 "47K" V 6600 3050 50  0000 C CNN
 F 2 "Resistors_SMD:R_0402" H 6650 2850 60  0001 C CNN
 F 3 "" H 6650 2850 60  0000 C CNN
+F 4 "ERJ-2RKF4702X" V 6650 2850 60  0001 C CNN "ManPartNo"
+F 5 "P47.0KLCT-ND" V 6650 2850 60  0001 C CNN "DistPartNo"
 	1    6650 2850
 	0    1    1    0
@@
 P 6650 2950
 F 0 "R6" V 6600 2800 50  0000 C CNN
-F 1 "R_Small" V 6600 3200 50  0000 C CNN
+F 1 "47K" V 6600 3150 50  0000 C CNN
 F 2 "Resistors_SMD:R_0402" H 6650 2950 60  0001 C CNN
 F 3 "" H 6650 2950 60  0000 C CNN
+F 4 "ERJ-2RKF4702X" V 6650 2950 60  0001 C CNN "ManPartNo"
+F 5 "P47.0KLCT-ND" V 6650 2950 60  0001 C CNN "DistPartNo"
 	1    6650 2950
 	0    1    1    0
@@
 P 5350 2850
 F 0 "R3" V 5300 2700 50  0000 C CNN
-F 1 "R_Small" V 5300 3100 50  0000 C CNN
+F 1 "47K" V 5300 3050 50  0000 C CNN
 F 2 "Resistors_SMD:R_0402" H 5350 2850 60  0001 C CNN
 F 3 "" H 5350 2850 60  0000 C CNN
+F 4 "ERJ-2RKF4702X" V 5350 2850 60  0001 C CNN "ManPartNo"
+F 5 "P47.0KLCT-ND" V 5350 2850 60  0001 C CNN "DistPartNo"
 	1    5350 2850
 	0    1    1    0
@@
 P 5350 2950
 F 0 "R5" V 5300 2800 50  0000 C CNN
-F 1 "R_Small" V 5300 3200 50  0000 C CNN
+F 1 "47K" V 5300 3150 50  0000 C CNN
 F 2 "Resistors_SMD:R_0402" H 5350 2950 60  0001 C CNN
 F 3 "" H 5350 2950 60  0000 C CNN
+F 4 "ERJ-2RKF4702X" V 5350 2950 60  0001 C CNN "ManPartNo"
+F 5 "P47.0KLCT-ND" V 5350 2950 60  0001 C CNN "DistPartNo"
 	1    5350 2950
 	0    1    1    0
@@
 F 2 "slocalization:SOT-363" H 6300 3400 60  0001 C CNN
 F 3 "" H 6300 3400 60  0000 C CNN
+F 4 "74LVC1G175GW,125" H 6300 3400 60  0001 C CNN "ManPartNo"
+F 5 "568-7761-1-ND" H 6300 3400 60  0001 C CNN "DistPartNo"
 	1    6300 3400
 	1    0    0    -1
@@
 F 2 "slocalization:SOT-363" H 6300 3900 60  0001 C CNN
 F 3 "" H 6300 3900 60  0000 C CNN
+F 4 "74LVC1G175GW,125" H 6300 3900 60  0001 C CNN "ManPartNo"
+F 5 "568-7761-1-ND" H 6300 3900 60  0001 C CNN "DistPartNo"
 	1    6300 3900
 	1    0    0    -1
@@
 P 5250 4450
 F 0 "R7" V 5300 4250 50  0000 L CNN
-F 1 "R_Small" V 5300 4550 50  0000 L CNN
+F 1 "47K" V 5300 4550 50  0000 L CNN
 F 2 "Resistors_SMD:R_0402" H 5250 4450 60  0001 C CNN
 F 3 "" H 5250 4450 60  0000 C CNN
+F 4 "ERJ-2RKF4702X" V 5250 4450 60  0001 C CNN "ManPartNo"
+F 5 "P47.0KLCT-ND" V 5250 4450 60  0001 C CNN "DistPartNo"
 	1    5250 4450
 	1    0    0    -1
@@
 P 5350 4450
 F 0 "R8" V 5400 4250 50  0000 L CNN
-F 1 "R_Small" V 5400 4550 50  0000 L CNN
+F 1 "47K" V 5400 4550 50  0000 L CNN
 F 2 "Resistors_SMD:R_0402" H 5350 4450 60  0001 C CNN
 F 3 "" H 5350 4450 60  0000 C CNN
+F 4 "ERJ-2RKF4702X" V 5350 4450 60  0001 C CNN "ManPartNo"
+F 5 "P47.0KLCT-ND" V 5350 4450 60  0001 C CNN "DistPartNo"
 	1    5350 4450
 	1    0    0    -1
@@
 P 5450 4450
 F 0 "R9" V 5500 4250 50  0000 L CNN
-F 1 "R_Small" V 5500 4550 50  0000 L CNN
+F 1 "47K" V 5500 4550 50  0000 L CNN
 F 2 "Resistors_SMD:R_0402" H 5450 4450 60  0001 C CNN
 F 3 "" H 5450 4450 60  0000 C CNN
+F 4 "ERJ-2RKF4702X" V 5450 4450 60  0001 C CNN "ManPartNo"
+F 5 "P47.0KLCT-ND" V 5450 4450 60  0001 C CNN "DistPartNo"
 	1    5450 4450
 	1    0    0    -1
@@
 P 5550 4450
 F 0 "R10" V 5600 4250 50  0000 L CNN
-F 1 "R_Small" V 5600 4550 50  0000 L CNN
+F 1 "47K" V 5600 4550 50  0000 L CNN
 F 2 "Resistors_SMD:R_0402" H 5550 4450 60  0001 C CNN
 F 3 "" H 5550 4450 60  0000 C CNN
+F 4 "ERJ-2RKF4702X" V 5550 4450 60  0001 C CNN "ManPartNo"
+F 5 "P47.0KLCT-ND" V 5550 4450 60  0001 C CNN "DistPartNo"
 	1    5550 4450
 	1    0    0    -1
@@
 F 2 "TO_SOT_Packages_SMD:SOT-353" H 2450 2750 60  0001 C CNN
 F 3 "" H 2450 2750 60  0000 C CNN
+F 4 "74LVC1G04GW,125" H 2450 2750 60  0001 C CNN "ManPartNo"
+F 5 "568-1579-1-ND" H 2450 2750 60  0001 C CNN "DistPartNo"
 	1    2450 2750
 	1    0    0    -1
@@
 P 10200 2550
 F 0 "C6" V 10150 2450 50  0000 C CNN
-F 1 "C_Small" V 10150 2750 50  0000 C CNN
+F 1 "100pF" V 10150 2750 50  0000 C CNN
 F 2 "Capacitors_SMD:C_0402" H 10200 2550 60  0001 C CNN
 F 3 "" H 10200 2550 60  0000 C CNN
+F 4 "GRM1555C1H101JA01J" V 10200 2550 60  0001 C CNN "ManPartNo"
+F 5 "490-7754-1-ND" V 10200 2550 60  0001 C CNN "DistPartNo"
 	1    10200 2550
 	0    1    1    0
@@
 P 10200 2700
 F 0 "C7" V 10150 2600 50  0000 C CNN
-F 1 "C_Small" V 10150 2900 50  0000 C CNN
+F 1 "100pF" V 10150 2900 50  0000 C CNN
 F 2 "Capacitors_SMD:C_0402" H 10200 2700 60  0001 C CNN
 F 3 "" H 10200 2700 60  0000 C CNN
+F 4 "GRM1555C1H101JA01J" V 10200 2700 60  0001 C CNN "ManPartNo"
+F 5 "490-7754-1-ND" V 10200 2700 60  0001 C CNN "DistPartNo"
 	1    10200 2700
 	0    1    1    0
@@
 P 4600 4050
 F 0 "R11" V 4550 3900 50  0000 C CNN
-F 1 "R_Small" V 4550 4300 50  0000 C CNN
+F 1 "DNP" V 4550 4250 50  0000 C CNN
 F 2 "Resistors_SMD:R_0402" H 4600 4050 60  0001 C CNN
 F 3 "" H 4600 4050 60  0000 C CNN
@@
 P 4600 4150
 F 0 "R12" V 4550 4000 50  0000 C CNN
-F 1 "R_Small" V 4550 4400 50  0000 C CNN
+F 1 "11K" V 4550 4350 50  0000 C CNN
 F 2 "Resistors_SMD:R_0402" H 4600 4150 60  0001 C CNN
 F 3 "" H 4600 4150 60  0000 C CNN
+F 4 "ERJ-2RKF1102X" V 4600 4150 60  0001 C CNN "ManPartNo"
+F 5 "P11.0KLCT-ND" V 4600 4150 60  0001 C CNN "DistPartNo"
 	1    4600 4150
 	0    1    1    0

Commit message: minor cosmetic fixes
Parts:
- removed C5: 100pF, Capacitors_SMD:C_0402, symbol C_Small
Connections:
- net at A1.1: now also U3.5 (RFC)
Changed lines of the file:
@@
-$EndComp
-$Comp
-L C_Small C5
-U 1 1 56C7AB0D
-P 10200 2250
-F 0 "C5" V 10150 2150 50  0000 C CNN
-F 1 "100pF" V 10150 2450 50  0000 C CNN
-F 2 "Capacitors_SMD:C_0402" H 10200 2250 60  0001 C CNN
-F 3 "" H 10200 2250 60  0000 C CNN
-F 4 "GRM1555C1H101JA01J" V 10200 2250 60  0001 C CNN "ManPartNo"
-F 5 "490-7754-1-ND" V 10200 2250 60  0001 C CNN "DistPartNo"
-	1    10200 2250
-	0    1    1    0
 $EndComp
 $Comp
@@
 	8850 1800 8850 1850
 Wire Wire Line
-	9850 2250 10100 2250
-Wire Wire Line
-	10300 2250 10600 2250
+	9850 2250 10600 2250
 Wire Wire Line
 	10600 2250 10600 2100
